Commit message: ScaledUpRobot

File: robot_description/urdf/DiffDriveScale_One.urdf (robot description, URDF)
Before this commit: robot Jeevan, 7 links, 6 joints
Links:
- link base_link: geometry collision box size=07.5 04 01; visual box size=07.5 04 01
- link camera_link: geometry collision box size=0.5 0.5 0.5; visual box size=0.5 0.5 0.5
- link caster: geometry collision sphere radius=0.81; visual sphere radius=0.81
- link laser: geometry collision sphere radius=.8; visual cylinder length=0.5 radius=0.5
- link wheel_left_link: geometry collision cylinder length=1 radius=1.5; visual cylinder length=1 radius=1.5
- link wheel_right_link: geometry collision cylinder length=1 radius=01.5; visual cylinder length=1 radius=01.5
Joints:
- joint base_joint: origin xyz=-0.15 0.0 0.15 rpy=0.0 0.0 0.0 -> xyz=1.5 0.0 01.5 rpy=0.0 0.0 0.0
- joint camera_joint: origin xyz=0.545 0 0.275 rpy=0 0 0 -> xyz=05.45 0 02.75 rpy=0 0 0
- joint caster_joint: origin xyz=0.45 0.0 0.076 rpy=0.0 0.0 0.0 -> xyz=04.5 0.0 0.76 rpy=0.0 0.0 0.0
- joint laser_joint: origin xyz=0.525 0.0 0.225 rpy=0.0 0.0 0.0 -> xyz=5.25 0.0 02.25 rpy=0.0 0.0 0.0
- joint wheel_left_joint: origin xyz=0. 0.25 0.15 rpy=-1.57 0.0 0.0 -> xyz=0. 02.5 01.5 rpy=-1.57 0.0 0.0
- joint wheel_right_joint: origin xyz=0 -0.25 0.15 rpy=-1.57 0.0 0.0 -> xyz=0 -02.5 01.5 rpy=-1.57 0.0 0.0
